Commit message: updated path names and added launch file

File: vehicles/alpha_follower.scn.xacro (robot description, xacro)
@@ -8,6 +8,6 @@
 -->
 <scenario xmlns:xacro="http://ros.org/wiki/xacro">
-    <xacro:include filename="$(find alpha_swarm_stonefish)/description/looks.scn.xacro"/>
-    <xacro:include filename="$(find alpha_swarm_stonefish)/description/materials.scn.xacro"/>
+    <xacro:include filename="$(find world_of_stonefish)/metadata/looks.scn.xacro"/>
+    <xacro:include filename="$(find world_of_stonefish)/metadata/materials.scn.xacro"/>
     <xacro:macro name="alpha_follower" params="xyz rpy robot_name">
         <robot name="${robot_name}" fixed="false" self_collisions="false">
@@ -15,9 +15,9 @@
                 <external_part name="Hull" type="model" physics="submerged" buoyant="false">
                     <physical>
-                        <mesh filename="hull_phy_reduced.obj" scale="1.0"/>
+                        <mesh filename="parts/body/hull_phy_reduced.obj" scale="1.0"/>
                         <origin rpy="0.0 0.0 0.0" xyz="0.0 0.0 0.0"/>
                     </physical>
                     <visual>
-                        <mesh filename="hull.obj" scale="1.0"/>
+                        <mesh filename="parts/body/hull.obj" scale="1.0"/>
                         <origin rpy="0.0 0.0 0.0" xyz="0.0 0.0 0.0"/>
                     </visual>
@@ -39,9 +39,9 @@
                 <external_part name="Mast" type="model" physics="submerged">
                     <physical>
-                        <mesh filename="mast.obj" scale="0.001"/>
+                        <mesh filename="parts/others/mast.obj" scale="0.001"/>
                         <origin rpy="-1.571 0.0 1.571"  xyz="-1.0 0.0 0.0"/>
                     </physical>
                     <visual>
-                        <mesh filename="mast.obj" scale="0.001"/>
+                        <mesh filename="parts/others/mast.obj" scale="0.001"/>
                         <origin rpy="-1.571 0.0 1.571" xyz="-1.0 0.0 0.0"/>
                     </visual>
@@ -52,9 +52,9 @@
                 <external_part name="ThrusterDuctSurge" type="model" physics="submerged" buoyant="false">
                     <physical>
-                        <mesh filename="duct.obj" scale="0.0015"/>
+                        <mesh filename="parts/thruster/duct.obj" scale="0.0015"/>
                         <origin rpy="0.0 1.571 0.0" xyz="-1.325 0.0 0.0"/>
                     </physical>
                     <visual>
-                        <mesh filename="duct.obj" scale="0.0015"/>
+                        <mesh filename="parts/thruster/duct.obj" scale="0.0015"/>
                         <origin rpy="0.0 1.571 0.0" xyz="-1.325 0.0 0.0"/>
                     </visual>
@@ -83,5 +83,5 @@
                 <specs thrust_coeff="0.4315" thrust_coeff_backward="0.3404" torque_coeff="0.01" max_rpm="3000.0"/>
                 <propeller diameter="0.08" right="true">
-                    <mesh filename="prop.obj" scale="1.0"/>
+                    <mesh filename="parts/thruster/prop.obj" scale="1.0"/>
                     <material name="Neutral"/>
                     <look name="white"/>
@@ -94,5 +94,5 @@
                 <specs thrust_coeff="0.4315" thrust_coeff_backward="0.3404" torque_coeff="0.01" max_rpm="3000.0"/>
                 <propeller diameter="0.08" right="true">
-                    <mesh filename="prop.obj" scale="1.0"/>
+                    <mesh filename="parts/thruster/prop.obj" scale="1.0"/>
                     <material name="Neutral"/>
                     <look name="white"/>
@@ -105,5 +105,5 @@
                 <specs thrust_coeff="0.4315" thrust_coeff_backward="0.3404" torque_coeff="0.01" max_rpm="3000.0"/>
                 <propeller diameter="0.08" right="true">
-                    <mesh filename="prop.obj" scale="1.0"/>
+                    <mesh filename="parts/thruster/prop.obj" scale="1.0"/>
                     <material name="Neutral"/>
                     <look name="white"/>
@@ -117,5 +117,5 @@
                 <propeller diameter="0.08" right="true">
                     <origin rpy="1.571 0.0 0.0" xyz="0.0 0.0 0.0"/>
-                    <mesh filename="prop.obj" scale="1.5"/>
+                    <mesh filename="parts/thruster/prop.obj" scale="1.5"/>
                     <material name="Neutral"/>
                     <look name="white"/>

File: vehicles/alpha_leader.scn.xacro (robot description, xacro)
@@ -8,6 +8,6 @@
 -->
 <scenario xmlns:xacro="http://ros.org/wiki/xacro">
-    <xacro:include filename="$(find alpha_swarm_stonefish)/description/looks.scn.xacro"/>
-    <xacro:include filename="$(find alpha_swarm_stonefish)/description/materials.scn.xacro"/>
+    <xacro:include filename="$(find world_of_stonefish)/metadata/looks.scn.xacro"/>
+    <xacro:include filename="$(find world_of_stonefish)/metadata/materials.scn.xacro"/>
     <xacro:macro name="alpha_leader" params="xyz rpy robot_name">
         <robot name="${robot_name}" fixed="false" self_collisions="false">
@@ -15,9 +15,9 @@
                 <external_part name="Hull" type="model" physics="submerged" buoyant="false">
                     <physical>
-                        <mesh filename="hull_phy_reduced.obj" scale="1.0"/>
+                        <mesh filename="parts/body/hull_phy_reduced.obj" scale="1.0"/>
                         <origin rpy="0.0 0.0 0.0" xyz="0.0 0.0 0.0"/>
                     </physical>
                     <visual>
-                        <mesh filename="hull.obj" scale="1.0"/>
+                        <mesh filename="parts/body/hull.obj" scale="1.0"/>
                         <origin rpy="0.0 0.0 0.0" xyz="0.0 0.0 0.0"/>
                     </visual>
@@ -39,9 +39,9 @@
                 <external_part name="Mast" type="model" physics="submerged">
                     <physical>
-                        <mesh filename="mast.obj" scale="0.001"/>
+                        <mesh filename="parts/others/mast.obj" scale="0.001"/>
                         <origin rpy="-1.571 0.0 1.571"  xyz="-1.0 0.0 0.0"/>
                     </physical>
                     <visual>
-                        <mesh filename="mast.obj" scale="0.001"/>
+                        <mesh filename="parts/others/mast.obj" scale="0.001"/>
                         <origin rpy="-1.571 0.0 1.571" xyz="-1.0 0.0 0.0"/>
                     </visual>
@@ -52,9 +52,9 @@
                 <external_part name="ThrusterDuctSurge" type="model" physics="submerged" buoyant="false">
                     <physical>
-                        <mesh filename="duct.obj" scale="0.0015"/>
+                        <mesh filename="parts/thruster/duct.obj" scale="0.0015"/>
                         <origin rpy="0.0 1.571 0.0" xyz="-1.325 0.0 0.0"/>
                     </physical>
                     <visual>
-                        <mesh filename="duct.obj" scale="0.0015"/>
+                        <mesh filename="parts/thruster/duct.obj" scale="0.0015"/>
                         <origin rpy="0.0 1.571 0.0" xyz="-1.325 0.0 0.0"/>
                     </visual>
@@ -83,5 +83,5 @@
                 <specs thrust_coeff="0.4315" thrust_coeff_backward="0.3404" torque_coeff="0.01" max_rpm="3000.0"/>
                 <propeller diameter="0.08" right="true">
-                    <mesh filename="prop.obj" scale="1.0"/>
+                    <mesh filename="parts/thruster/prop.obj" scale="1.0"/>
                     <material name="Neutral"/>
                     <look name="white"/>
@@ -94,5 +94,5 @@
                 <specs thrust_coeff="0.4315" thrust_coeff_backward="0.3404" torque_coeff="0.01" max_rpm="3000.0"/>
                 <propeller diameter="0.08" right="true">
-                    <mesh filename="prop.obj" scale="1.0"/>
+                    <mesh filename="parts/thruster/prop.obj" scale="1.0"/>
                     <material name="Neutral"/>
                     <look name="white"/>
@@ -105,5 +105,5 @@
                 <specs thrust_coeff="0.4315" thrust_coeff_backward="0.3404" torque_coeff="0.01" max_rpm="3000.0"/>
                 <propeller diameter="0.08" right="true">
-                    <mesh filename="prop.obj" scale="1.0"/>
+                    <mesh filename="parts/thruster/prop.obj" scale="1.0"/>
                     <material name="Neutral"/>
                     <look name="white"/>
@@ -117,5 +117,5 @@
                 <propeller diameter="0.08" right="true">
                     <origin rpy="1.571 0.0 0.0" xyz="0.0 0.0 0.0"/>
-                    <mesh filename="prop.obj" scale="1.5"/>
+                    <mesh filename="parts/thruster/prop.obj" scale="1.5"/>
                     <material name="Neutral"/>
                     <look name="white"/>

File: vehicles/alpha_std.scn.xacro (robot description, xacro)
@@ -8,6 +8,6 @@
 -->
 <scenario xmlns:xacro="http://ros.org/wiki/xacro">
-    <xacro:include filename="$(find alpha_std_stonefish)/description/looks.scn.xacro"/>
-    <xacro:include filename="$(find alpha_std_stonefish)/description/materials.scn.xacro"/>
+    <xacro:include filename="$(find world_of_stonefish)/metadata/looks.scn.xacro"/>
+    <xacro:include filename="$(find world_of_stonefish)/metadata/materials.scn.xacro"/>
     <xacro:macro name="alpha_std" params="xyz rpy robot_name">
         <robot name="${robot_name}" fixed="false" self_collisions="false">
@@ -15,9 +15,9 @@
                 <external_part name="Hull" type="model" physics="submerged" buoyant="false">
                     <physical>
-                        <mesh filename="hull_phy_reduced.obj" scale="1.0"/>
+                        <mesh filename="parts/body/hull_phy_reduced.obj" scale="1.0"/>
                         <origin rpy="0.0 0.0 0.0" xyz="0.0 0.0 0.0"/>
                     </physical>
                     <visual>
-                        <mesh filename="hull.obj" scale="1.0"/>
+                        <mesh filename="parts/body/hull.obj" scale="1.0"/>
                         <origin rpy="0.0 0.0 0.0" xyz="0.0 0.0 0.0"/>
                     </visual>
@@ -39,9 +39,9 @@
                 <external_part name="Mast" type="model" physics="submerged">
                     <physical>
-                        <mesh filename="mast.obj" scale="0.001"/>
+                        <mesh filename="parts/others/mast.obj" scale="0.001"/>
                         <origin rpy="-1.571 0.0 1.571"  xyz="-1.0 0.0 0.0"/>
                     </physical>
                     <visual>
-                        <mesh filename="mast.obj" scale="0.001"/>
+                        <mesh filename="parts/others/mast.obj" scale="0.001"/>
                         <origin rpy="-1.571 0.0 1.571" xyz="-1.0 0.0 0.0"/>
                     </visual>
@@ -52,9 +52,9 @@
                 <external_part name="ThrusterDuctSurge" type="model" physics="submerged" buoyant="false">
                     <physical>
-                        <mesh filename="duct.obj" scale="0.0015"/>
+                        <mesh filename="parts/thruster/duct.obj" scale="0.0015"/>
                         <origin rpy="0.0 1.571 0.0" xyz="-1.325 0.0 0.0"/>
                     </physical>
                     <visual>
-                        <mesh filename="duct.obj" scale="0.0015"/>
+                        <mesh filename="parts/thruster/duct.obj" scale="0.0015"/>
                         <origin rpy="0.0 1.571 0.0" xyz="-1.325 0.0 0.0"/>
                     </visual>
@@ -83,5 +83,5 @@
                 <specs thrust_coeff="0.4315" thrust_coeff_backward="0.3404" torque_coeff="0.01" max_rpm="3000.0"/>
                 <propeller diameter="0.08" right="true">
-                    <mesh filename="prop.obj" scale="1.0"/>
+                    <mesh filename="parts/thruster/prop.obj" scale="1.0"/>
                     <material name="Neutral"/>
                     <look name="white"/>
@@ -94,5 +94,5 @@
                 <specs thrust_coeff="0.4315" thrust_coeff_backward="0.3404" torque_coeff="0.01" max_rpm="3000.0"/>
                 <propeller diameter="0.08" right="true">
-                    <mesh filename="prop.obj" scale="1.0"/>
+                    <mesh filename="parts/thruster/prop.obj" scale="1.0"/>
                     <material name="Neutral"/>
                     <look name="white"/>
@@ -105,5 +105,5 @@
                 <specs thrust_coeff="0.4315" thrust_coeff_backward="0.3404" torque_coeff="0.01" max_rpm="3000.0"/>
                 <propeller diameter="0.08" right="true">
-                    <mesh filename="prop.obj" scale="1.0"/>
+                    <mesh filename="parts/thruster/prop.obj" scale="1.0"/>
                     <material name="Neutral"/>
                     <look name="white"/>
@@ -117,5 +117,5 @@
                 <propeller diameter="0.08" right="true">
                     <origin rpy="1.571 0.0 0.0" xyz="0.0 0.0 0.0"/>
-                    <mesh filename="prop.obj" scale="1.5"/>
+                    <mesh filename="parts/thruster/prop.obj" scale="1.5"/>
                     <material name="Neutral"/>
                     <look name="white"/>

File: world/ocean.scn.xacro (robot description, xacro)
@@ -9,5 +9,5 @@
 <scenario xmlns:xacro="http://ros.org/wiki/xacro">
     <xacro:arg name="robot_name" default="changeme"/>
-    <xacro:include filename="$(find alpha_std_stonefish)/description/alpha_std.scn.xacro"/>
+    <xacro:include filename="$(find world_of_stonefish)/vehicles/alpha_std.scn.xacro"/>
     <xacro:alpha_std robot_name="$(arg robot_name)" xyz="0.0 0.0 0.0" rpy="0.0 0.0 0.0"/>
     <environment>
@@ -32,9 +32,9 @@
     <static name="Bottom" type="model">
         <physical>
-            <mesh filename="flat_terrain.obj" scale="2.0" convex="true"/>
+            <mesh filename="objects/flat_terrain.obj" scale="2.0" convex="true"/>
             <origin xyz="0.0 0.0 0.0" rpy="0.0 0.0 0.0"/>
         </physical>
         <visual>
-            <mesh filename="flat_terrain.obj" scale="2.0"/>
+            <mesh filename="objects/flat_terrain.obj" scale="2.0"/>
             <origin xyz="0.0 0.0 0.0" rpy="0.0 0.0 0.0"/>
         </visual>

File: world/ocean_multi_agent.scn.xacro (robot description, xacro)
@@ -8,9 +8,9 @@
 -->
 <scenario xmlns:xacro="http://ros.org/wiki/xacro">
-    <xacro:include filename="$(find alpha_sci_stonefish)/description/alpha_sci.scn.xacro"/>
-    <xacro:alpha_sci robot_name="bill" xyz="0.0 0.0 0.0" rpy="0.0 0.0 0.0"/>
-    <xacro:alpha_sci robot_name="lin" xyz="5.0 0.0 0.0" rpy="0.0 0.0 0.0"/>
-    <xacro:alpha_sci robot_name="emir" xyz="5.0 5.0 0.0" rpy="0.0 0.0 0.0"/>
-    <xacro:alpha_sci robot_name="mingxi" xyz="0.0 5.0 0.0" rpy="0.0 0.0 0.0"/>
+    <xacro:include filename="$(find world_of_stonefish)/vehicles/alpha_std.scn.xacro"/>
+    <xacro:alpha_std robot_name="bill" xyz="0.0 0.0 0.0" rpy="0.0 0.0 0.0"/>
+    <xacro:alpha_std robot_name="lin" xyz="5.0 0.0 0.0" rpy="0.0 0.0 0.0"/>
+    <xacro:alpha_std robot_name="emir" xyz="5.0 5.0 0.0" rpy="0.0 0.0 0.0"/>
+    <xacro:alpha_std robot_name="mingxi" xyz="0.0 5.0 0.0" rpy="0.0 0.0 0.0"/>
     <environment>
         <ned latitude="41" longitude="71"/>
@@ -29,9 +29,9 @@
     <static name="Bottom" type="model">
         <physical>
-            <mesh filename="seabed.obj" scale="2.0" convex="false"/>
+            <mesh filename="objects/seabed.obj" scale="2.0" convex="false"/>
             <origin xyz="0.0 0.0 0.0" rpy="0.0 0.0 0.0"/>
         </physical>
         <visual>
-            <mesh filename="seabed.obj" scale="2.0"/>
+            <mesh filename="objects/seabed.obj" scale="2.0"/>
             <origin xyz="0.0 0.0 0.0" rpy="0.0 0.0 0.0"/>
         </visual>

File: world/ocean_swarm.scn.xacro (robot description, xacro)
@@ -8,6 +8,6 @@
 -->
 <scenario xmlns:xacro="http://ros.org/wiki/xacro">
-    <xacro:include filename="$(find alpha_swarm_stonefish)/description/alpha_leader.scn.xacro"/>
-    <xacro:include filename="$(find alpha_swarm_stonefish)/description/alpha_follower.scn.xacro"/>
+    <xacro:include filename="$(find world_of_stonefish)/vehicles/alpha_leader.scn.xacro"/>
+    <xacro:include filename="$(find world_of_stonefish)/vehicles/alpha_follower.scn.xacro"/>
     <xacro:alpha_leader robot_name="leader" xyz="0.0 0.0 0.0" rpy="0.0 0.0 0.0"/>
     <xacro:alpha_follower robot_name="follower" xyz="-20.0 0.0 0.0" rpy="0.0 0.0 0.0"/>
@@ -28,9 +28,9 @@
     <static name="Bottom" type="model">
         <physical>
-            <mesh filename="seabed.obj" scale="2.0" convex="false"/>
+            <mesh filename="objects/seabed.obj" scale="2.0" convex="false"/>
             <origin xyz="0.0 0.0 0.0" rpy="0.0 0.0 0.0"/>
         </physical>
         <visual>
-            <mesh filename="seabed.obj" scale="2.0"/>
+            <mesh filename="objects/seabed.obj" scale="2.0"/>
             <origin xyz="0.0 0.0 0.0" rpy="0.0 0.0 0.0"/>
         </visual>

File: world/tank.scn.xacro (robot description, xacro)
@@ -9,6 +9,6 @@
 <scenario xmlns:xacro="http://ros.org/wiki/xacro">
     <xacro:arg name="robot_name" default="changeme"/>
-    <xacro:include filename="$(find alpha_std_stonefish)/description/alpha_std.scn.xacro"/>
-    <xacro:alpha_sci robot_name="$(arg robot_name)" xyz="0.0 0.0 0.0" rpy="0.0 0.0 0.0"/>
+    <xacro:include filename="$(find world_of_stonefish)/vehicles/alpha_std.scn.xacro"/>
+    <xacro:alpha_std robot_name="$(arg robot_name)" xyz="0.0 0.0 0.0" rpy="0.0 0.0 0.0"/>
     <environment>
         <ned latitude="41.7777" longitude="3.0333"/>
@@ -27,9 +27,9 @@
     <static name="tank" type="model">
         <physical>
-            <mesh filename="tank.obj" scale="1.0" convex="false"/>
+            <mesh filename="objects/tank.obj" scale="1.0" convex="false"/>
             <origin xyz="0.0 0.0 0.0" rpy="0.0 0.0 0.0"/>
         </physical>
         <visual>
-            <mesh filename="tank.obj" scale="1.0"/>
+            <mesh filename="objects/tank.obj" scale="1.0"/>
             <origin xyz="0.0 0.0 0.0" rpy="0.0 0.0 0.0"/>
         </visual>
