Commit message: feat:reduced iceberg scale

File: vehicles/wamv.scn.xacro (robot description, xacro)
@@ -59,5 +59,5 @@
                     <cg xyz=" 0.0 0 1.0" rpy="0.0 0.0 0.0"/>
                 </external_part>
-                <external_part name="thrusterPort" type="model" physics="submerged" buoyant="false">
+                <!-- <external_part name="thrusterPort" type="model" physics="submerged" buoyant="false">
                     <physical>
                         <mesh filename="$(find world_of_stonefish)/data/parts/thruster/wamv_propeller.obj" scale="0.5"/>
@@ -84,5 +84,5 @@
                     <look name="black"/>
                     <compound_transform rpy="0.0 0.0 0.0" xyz="0.0 0.0 0.0"/>
-                </external_part>
+                </external_part> -->
             </base_link>
             <!-- the actual base frame  -->
@@ -106,5 +106,5 @@
                     <mesh filename="$(find world_of_stonefish)/data/parts/thruster/wamv_propeller.obj" scale="0.5"/>
                     <material name="Neutral"/>
-                    <look name="white"/>
+                    <look name="black"/>
                 </propeller>
                 <ros_subscriber topic="/${robot_name}/control/thruster/port"/>
@@ -117,5 +117,5 @@
                     <mesh filename="$(find world_of_stonefish)/data/parts/thruster/wamv_propeller.obj" scale="0.5"/>
                     <material name="Neutral"/>
-                    <look name="white"/>
+                    <look name="black"/>
                 </propeller>
                 <ros_subscriber topic="/${robot_name}/control/thruster/starboard"/>
@@ -199,8 +199,14 @@
             </sensor> -->
             <sensor name="Cam" rate="10.0" type="camera">
-                <specs resolution_x="800" resolution_y="600" horizontal_fov="60.0"/>
-                <origin xyz="0.0 0.0 -0.3" rpy="-1.57 3.14 4.71"/>
-                <link name="Base"/>
-                <ros_publisher topic="/${robot_name}/camera/stonefish/data"/>
+                <specs resolution_x="800" resolution_y="600" horizontal_fov="120.0"/>
+                <origin xyz="0.0 0.0 -1" rpy="-1.57 3.14 0"/>
+                <link name="Base"/>
+                <ros_publisher topic="/${robot_name}/camera/stonefish/side/data"/>
+            </sensor>
+            <sensor name="Cam_front" rate="10.0" type="camera">
+                <specs resolution_x="800" resolution_y="600" horizontal_fov="120.0"/>
+                <origin xyz="-1. 0.0 -1" rpy="-1.57 3.14 4.71"/>
+                <link name="Base"/>
+                <ros_publisher topic="/${robot_name}/camera/stonefish/front/data"/>
             </sensor>
             <world_transform rpy="${rpy}" xyz="${xyz}"/>

File: world/iceberg.scn.xacro (robot description, xacro)
@@ -12,10 +12,10 @@
     <static name="iceberg" type="model">
         <physical>
-            <mesh filename="objects/iceberg_01.obj" scale="1.0" convex="false"/>
-            <origin xyz="-20 -15 0.0" rpy="0.0 0.0 0.0"/>
+            <mesh filename="objects/iceberg_01.obj" scale="0.5" convex="false"/>
+            <origin xyz="-40 10 0.0" rpy="0.0 0.0 0.0"/>
         </physical>
         <visual>
-            <mesh filename="objects/iceberg_01.obj" scale="1.0"/>
-            <origin xyz="-20 -15 0.0" rpy="0.0 0.0 0.0"/>
+            <mesh filename="objects/iceberg_01.obj" scale="0.5"/>
+            <origin xyz="-40 10 0.0" rpy="0.0 0.0 0.0"/>
         </visual>
         <material name="Ice"/>

File: world/ocean_rise.scn.xacro (robot description, xacro)
@@ -9,9 +9,9 @@
 <scenario xmlns:xacro="http://ros.org/wiki/xacro">
     <xacro:arg name="robot_name" default="changeme"/>
-    <!-- <xacro:include filename="$(find world_of_stonefish)/world/iceberg.scn.xacro"/> -->
+    <xacro:include filename="$(find world_of_stonefish)/world/iceberg.scn.xacro"/>
     <xacro:include filename="$(find world_of_stonefish)/vehicles/alpha_rise.scn.xacro"/>
-    <!-- <xacro:include filename="$(find world_of_stonefish)/vehicles/wamv.scn.xacro"/> -->
+    <xacro:include filename="$(find world_of_stonefish)/vehicles/wamv.scn.xacro"/>
     <xacro:alpha_rise robot_name="alpha_rise" xyz="0.0 0.0 0.0" rpy="0.0 0.0 0.0"/>
-    <!-- <xacro:wamv robot_name="wamv" xyz="0.0 10.0 0.0" rpy="0.0 0.0 0.0"/> -->
+    <xacro:wamv robot_name="wamv" xyz="0.0 5.0 0.0" rpy="0.0 0.0 0.0"/>
     <environment>
         <ned latitude="41" longitude="-71"/>
