Commit message: added ocean rise scenario

File: vehicles/alpha_rise.scn.xacro (robot description, xacro)
@@ -15,9 +15,9 @@
                 <external_part name="Hull" type="model" physics="submerged" buoyant="false">
                     <physical>
-                        <mesh filename="parts/body/hull_phy_reduced.obj" scale="1.0"/>
+                        <mesh filename="parts/body/hull_mk2_reduced.obj" scale="0.001"/>
                         <origin rpy="0.0 0.0 0.0" xyz="0.0 0.0 0.0"/>
                     </physical>
                     <visual>
-                        <mesh filename="parts/body/hull.obj" scale="1.0"/>
+                        <mesh filename="parts/body/hull_mk2_visual.obj" scale="0.001"/>
                         <origin rpy="0.0 0.0 0.0" xyz="0.0 0.0 0.0"/>
                     </visual>
@@ -188,4 +188,5 @@
             </sensor> -->
             <world_transform rpy="${rpy}" xyz="${xyz}"/>
+            <!-- <world_transform xyz="0.0 0.0 0.0" rpy="0.0 0.0 0.0"/> -->
         </robot>
     </xacro:macro>

File: world/ocean_rise.scn.xacro (robot description, xacro)
@@ -10,5 +10,5 @@
     <xacro:arg name="robot_name" default="changeme"/>
     <xacro:include filename="$(find world_of_stonefish)/vehicles/$(arg robot_name).scn.xacro"/>
-    <xacro:alpha_std robot_name="$(arg robot_name)" xyz="0.0 0.0 0.0" rpy="0.0 0.0 0.0"/>
+    <xacro:alpha_rise robot_name="$(arg robot_name)" xyz="0.0 0.0 0.0" rpy="0.0 0.0 0.0"/>
     <environment>
         <ned latitude="41" longitude="-71"/>

Commit message: changed thruster locations

File: vehicles/alpha_rise.scn.xacro (robot description, xacro)
@@ -16,9 +16,9 @@
                     <physical>
                         <mesh filename="parts/body/hull_mk2_reduced.obj" scale="0.001"/>
-                        <origin rpy="0.0 0.0 0.0" xyz="0.0 0.0 0.0"/>
+                        <origin rpy="1.5707 0.0 0.0" xyz="0.0 0.0 0.0"/>
                     </physical>
                     <visual>
                         <mesh filename="parts/body/hull_mk2_visual.obj" scale="0.001"/>
-                        <origin rpy="0.0 0.0 0.0" xyz="0.0 0.0 0.0"/>
+                        <origin rpy="1.5707 0.0 0.0" xyz="0.0 0.0 0.0"/>
                     </visual>
                     <material name="Vehicle"/>
@@ -53,9 +53,9 @@
                     <physical>
                         <mesh filename="parts/thruster/duct.obj" scale="0.0015"/>
-                        <origin rpy="0.0 1.571 0.0" xyz="-1.325 0.0 0.0"/>
+                        <origin rpy="0.0 1.571 0.0" xyz="-1.4 0.0 0.0"/>
                     </physical>
                     <visual>
                         <mesh filename="parts/thruster/duct.obj" scale="0.0015"/>
-                        <origin rpy="0.0 1.571 0.0" xyz="-1.325 0.0 0.0"/>
+                        <origin rpy="0.0 1.571 0.0" xyz="-1.4 0.0 0.0"/>
                     </visual>
                     <material name="Neutral"/>
@@ -80,5 +80,5 @@
             <actuator name="ThrusterSwayBow" type="thruster">
                 <link name="Base"/>
-                <origin rpy="0.0 0.0 1.5707963" xyz="-0.18 0.0 0.0"/>
+                <origin rpy="0.0 0.0 1.5707963" xyz="-0.06 0.0 0.0"/>
                 <specs thrust_coeff="0.4315" thrust_coeff_backward="0.3404" torque_coeff="0.01" max_rpm="3000.0"/>
                 <propeller diameter="0.08" right="true">
@@ -91,5 +91,5 @@
             <actuator name="ThrusterHeaveStern" type="thruster">
                 <link name="Base"/>
-                <origin rpy="0.0 -1.571 0.0" xyz="-1.0956 0.0 0.0"/>
+                <origin rpy="0.0 -1.571 0.0" xyz="-0.9604 0.0 0.0"/>
                 <specs thrust_coeff="0.4315" thrust_coeff_backward="0.3404" torque_coeff="0.01" max_rpm="3000.0"/>
                 <propeller diameter="0.08" right="true">
@@ -103,5 +103,5 @@
             <actuator name="ThrusterHeaveBow" type="thruster">
                 <link name="Base"/>
-                <origin rpy="0.0 -1.571 0.0" xyz="-0.2857 0.0 0.0"/>
+                <origin rpy="0.0 -1.571 0.0" xyz="-0.185 0.0 0.0"/>
                 <specs thrust_coeff="0.4315" thrust_coeff_backward="0.3404" torque_coeff="0.01" max_rpm="3000.0"/>
                 <propeller diameter="0.08" right="true">
@@ -115,5 +115,5 @@
             <actuator name="ThrusterSurge" type="thruster">
                 <link name="Base"/>
-                <origin rpy="0.0 0.0 0.0" xyz="-1.325 0.0 0.0"/>
+                <origin rpy="0.0 0.0 0.0" xyz="-1.4 0.0 0.0"/>
                 <specs thrust_coeff="1.7568" thrust_coeff_backward="1.0882" torque_coeff="0.01" max_rpm="3000.0"/>
                 <propeller diameter="0.08" right="true">

Commit message: adjusted alpha rise thruster position

File: vehicles/alpha_rise.scn.xacro (robot description, xacro)
@@ -24,5 +24,5 @@
                     <material name="Vehicle"/>
                     <look name="yellow"/>
-                    <mass value="39.0"/>
+                    <mass value="38.7"/>
                     <inertia xyz="1.0 10.0 10.0"/>
                     <compound_transform rpy="0.0 0.0 0.0" xyz="0.0 0.0 0.0"/>
@@ -53,9 +53,9 @@
                     <physical>
                         <mesh filename="parts/thruster/duct.obj" scale="0.0015"/>
-                        <origin rpy="0.0 1.571 0.0" xyz="-1.4 0.0 0.0"/>
+                        <origin rpy="0.0 1.571 0.0" xyz="-1.5 0.0 0.0"/>
                     </physical>
                     <visual>
                         <mesh filename="parts/thruster/duct.obj" scale="0.0015"/>
-                        <origin rpy="0.0 1.571 0.0" xyz="-1.4 0.0 0.0"/>
+                        <origin rpy="0.0 1.571 0.0" xyz="-1.5 0.0 0.0"/>
                     </visual>
                     <material name="Neutral"/>
@@ -80,5 +80,5 @@
             <actuator name="ThrusterSwayBow" type="thruster">
                 <link name="Base"/>
-                <origin rpy="0.0 0.0 1.5707963" xyz="-0.06 0.0 0.0"/>
+                <origin rpy="0.0 0.0 1.5707963" xyz="-0.2295 0.0 0.0"/>
                 <specs thrust_coeff="0.4315" thrust_coeff_backward="0.3404" torque_coeff="0.01" max_rpm="3000.0"/>
                 <propeller diameter="0.08" right="true">
@@ -91,5 +91,5 @@
             <actuator name="ThrusterHeaveStern" type="thruster">
                 <link name="Base"/>
-                <origin rpy="0.0 -1.571 0.0" xyz="-0.9604 0.0 0.0"/>
+                <origin rpy="0.0 -1.571 0.0" xyz="-1.13 0.0 0.0"/>
                 <specs thrust_coeff="0.4315" thrust_coeff_backward="0.3404" torque_coeff="0.01" max_rpm="3000.0"/>
                 <propeller diameter="0.08" right="true">
@@ -103,5 +103,5 @@
             <actuator name="ThrusterHeaveBow" type="thruster">
                 <link name="Base"/>
-                <origin rpy="0.0 -1.571 0.0" xyz="-0.185 0.0 0.0"/>
+                <origin rpy="0.0 -1.571 0.0" xyz="-0.3545 0.0 0.0"/>
                 <specs thrust_coeff="0.4315" thrust_coeff_backward="0.3404" torque_coeff="0.01" max_rpm="3000.0"/>
                 <propeller diameter="0.08" right="true">
@@ -115,5 +115,5 @@
             <actuator name="ThrusterSurge" type="thruster">
                 <link name="Base"/>
-                <origin rpy="0.0 0.0 0.0" xyz="-1.4 0.0 0.0"/>
+                <origin rpy="0.0 0.0 0.0" xyz="-1.5 0.0 0.0"/>
                 <specs thrust_coeff="1.7568" thrust_coeff_backward="1.0882" torque_coeff="0.01" max_rpm="3000.0"/>
                 <propeller diameter="0.08" right="true">

Commit message: tested rudder in alpha_rise_auv

File: vehicles/alpha_rise.scn.xacro (robot description, xacro)
@@ -126,4 +126,17 @@
                 <ros_subscriber topic="/${robot_name}/control/thruster/surge"/>
             </actuator>
+            <actuator name="Rudder" type="rudder">
+                <link name="Base"/>
+                <!-- a manual angle -->
+                <!-- <origin rpy="0.0 0.0 0.2" xyz="0.0 0.0 0.0"/>  -->
+                <origin rpy="0.0 0.0 0.0" xyz="0.0 0.0 0.0"/>
+                <specs drag_coeff="1.0" lift_coeff="3.0" max_angle="0.6" inverted="false" area="0.06"/>
+                <visual>
+                    <mesh filename="parts/others/rudder.obj" scale="0.002"/>
+                    <material name="Neutral"/>
+                    <look name="black"/>
+                    <origin rpy="-1.571 1.571 0.3" xyz="-1.2 0.0 0.2"/>
+                </visual>
+            </actuator>
             <sensor name="pressure" type="pressure" rate="5.0">
                 <link name="Base"/>

File: world/ocean.scn.xacro (robot description, xacro)
@@ -15,5 +15,5 @@
         <ocean>
             <water density="1031.0" jerlov="0.2"/>
-            <waves height="0.0"/>
+            <!-- <waves height="0.0"/> -->
             <particles enabled="true"/>
             <current type="uniform">

Commit message: updated rise thruster to match reality

File: vehicles/alpha_rise.scn.xacro (robot description, xacro)
@@ -91,5 +91,5 @@
             <actuator name="ThrusterHeaveStern" type="thruster">
                 <link name="Base"/>
-                <origin rpy="0.0 -1.571 0.0" xyz="-1.13 0.0 0.0"/>
+                <origin rpy="0.0 1.571 0.0" xyz="-1.13 0.0 0.0"/>
                 <specs thrust_coeff="0.4315" thrust_coeff_backward="0.3404" torque_coeff="0.01" max_rpm="3000.0"/>
                 <propeller diameter="0.08" right="true">
@@ -103,5 +103,5 @@
             <actuator name="ThrusterHeaveBow" type="thruster">
                 <link name="Base"/>
-                <origin rpy="0.0 -1.571 0.0" xyz="-0.3545 0.0 0.0"/>
+                <origin rpy="0.0 1.571 0.0" xyz="-0.3545 0.0 0.0"/>
                 <specs thrust_coeff="0.4315" thrust_coeff_backward="0.3404" torque_coeff="0.01" max_rpm="3000.0"/>
                 <propeller diameter="0.08" right="true">
@@ -126,9 +126,9 @@
                 <ros_subscriber topic="/${robot_name}/control/thruster/surge"/>
             </actuator>
-            <actuator name="Rudder" type="rudder">
-                <link name="Base"/>
+            <!-- <actuator name="Rudder" type="rudder">
+                <link name="Base"/> -->
                 <!-- a manual angle -->
                 <!-- <origin rpy="0.0 0.0 0.2" xyz="0.0 0.0 0.0"/>  -->
-                <origin rpy="0.0 0.0 0.0" xyz="0.0 0.0 0.0"/>
+                <!-- <origin rpy="0.0 0.0 0.0" xyz="0.0 0.0 0.0"/>
                 <specs drag_coeff="1.0" lift_coeff="3.0" max_angle="0.6" inverted="false" area="0.06"/>
                 <visual>
@@ -138,5 +138,5 @@
                     <origin rpy="-1.571 1.571 0.3" xyz="-1.2 0.0 0.2"/>
                 </visual>
-            </actuator>
+            </actuator> -->
             <sensor name="pressure" type="pressure" rate="5.0">
                 <link name="Base"/>

Commit message: feat:added msis

File: vehicles/alpha_rise.scn.xacro (robot description, xacro)
@@ -126,9 +126,10 @@
                 <ros_subscriber topic="/${robot_name}/control/thruster/surge"/>
             </actuator>
+<!--
             <actuator name="Rudder" type="rudder">
-                <link name="Base"/>
+                <link name="Base"/> -->
                 <!-- a manual angle -->
                 <!-- <origin rpy="0.0 0.0 0.2" xyz="0.0 0.0 0.0"/>  -->
-                <origin rpy="0.0 0.0 0.0" xyz="0.0 0.0 0.0"/>
+                <!-- <origin rpy="0.0 0.0 0.0" xyz="0.0 0.0 0.0"/>
                 <specs drag_coeff="1.0" lift_coeff="3.0" max_angle="0.6" inverted="false" area="0.06"/>
                 <visual>
@@ -138,5 +139,5 @@
                     <origin rpy="-1.571 1.571 0.3" xyz="-1.2 0.0 0.2"/>
                 </visual>
-            </actuator>
+            </actuator> -->
             <sensor name="pressure" type="pressure" rate="5.0">
                 <link name="Base"/>
@@ -191,4 +192,13 @@
                 <ros_publisher topic="/${robot_name}/msis/data"/>
             </sensor> -->
+            <sensor name="MSIS" type="msis">
+                <specs step="1" bins="100" horizontal_beam_width="2.0" vertical_beam_width="30.0"/>
+                <settings range_min="0.5" range_max="50.0" rotation_min="-180.0" rotation_max="180.0" gain="1.5"/>
+                <noise multiplicative="0.02" additive="0.03"/>
+                <display colormap="hot"/>
+                <origin xyz="0.0 0.0 0.0" rpy="-1.57 3.14 4.71"/>
+                <ros_publisher topic="/${robot_name}/msis/stonefish/data"/>
+                <link name="Base"/>
+            </sensor>
             <!-- <sensor name="FLS" type="fls">
                 <specs beams="512" bins="250" horizontal_fov="120.0" vertical_fov="15.0"/>

Commit message: fix:tf of msis steonfish

File: vehicles/alpha_rise.scn.xacro (robot description, xacro)
@@ -199,5 +199,6 @@
                 <noise multiplicative="0.002" additive="0.003"/>
                 <display colormap="hot"/>
-                <origin xyz="0.0 0.0 0.0" rpy="-1.57 3.14 4.71"/>
+                <origin xyz="0.0 0.0 0.0" rpy="1.57 0 0"/>
+                <!-- <origin xyz="0.0 0.0 0.0" rpy="1.57 3.14 4.71"/> -->
                 <ros_publisher topic="/${robot_name}/msis/stonefish/data"/>
                 <link name="Base"/>

Commit message: fix:tf msis

File: vehicles/alpha_rise.scn.xacro (robot description, xacro)
@@ -199,5 +199,5 @@
                 <noise multiplicative="0.002" additive="0.003"/>
                 <display colormap="hot"/>
-                <origin xyz="0.0 0.0 0.0" rpy="1.57 0 0"/>
+                <origin xyz="0.0 0.0 0.0" rpy="1.57 0 1.57"/>
                 <!-- <origin xyz="0.0 0.0 0.0" rpy="1.57 3.14 4.71"/> -->
                 <ros_publisher topic="/${robot_name}/msis/stonefish/data"/>

Commit message: updated stonefish file for alpha_rise to make thruster and imu matching the real orientation. commented out iceberg and wam-v in ocean_rise.scn for alpha testing

File: vehicles/alpha_rise.scn.xacro (robot description, xacro)
@@ -80,5 +80,5 @@
             <actuator name="ThrusterSwayBow" type="thruster">
                 <link name="Base"/>
-                <origin rpy="0.0 0.0 1.5707963" xyz="-0.2295 0.0 0.0"/>
+                <origin rpy="0.0 0.0 -1.5707963" xyz="-0.2295 0.0 0.0"/>
                 <specs thrust_coeff="0.4315" thrust_coeff_backward="0.3404" torque_coeff="0.01" max_rpm="3000.0"/>
                 <propeller diameter="0.08" right="true">
@@ -153,11 +153,11 @@
                 <specs beam_angle="30.0"/>
                 <range velocity="9.0 9.0 9.0" altitude_min="0.2" altitude_max="200.0"/>
-                <noise velocity="0.015" altitude="0.001"/>
+                <noise velocity="0.01" altitude="0.001"/>
                 <ros_publisher topic="/${robot_name}/dvl/twist" altitude_topic="/${robot_name}/dvl/altitude"/>
             </sensor>
             <sensor name="imu_sf" type="imu" rate="20.0">
                 <link name="Base"/>
-                <origin rpy="3.1415926 0.0 0.0" xyz="-0.65 0.0 -0.05"/>
-                <noise angle="0.001 0.001 0.005" angular_velocity="0.005" yaw_drift="0.001" linear_acceleration="0.001"/>
+                <origin rpy="0.0 0.0 3.1415926" xyz="-0.65 0.0 -0.05"/>
+                <noise angle="0.0001 0.0001 0.0001" angular_velocity="0.0001" yaw_drift="0.0001" linear_acceleration="0.0001"/>
                 <ros_publisher topic="/${robot_name}/imu/stonefish/data"/>
             </sensor>

File: world/ocean_rise.scn.xacro (robot description, xacro)
@@ -9,9 +9,9 @@
 <scenario xmlns:xacro="http://ros.org/wiki/xacro">
     <xacro:arg name="robot_name" default="changeme"/>
-    <xacro:include filename="$(find world_of_stonefish)/world/iceberg.scn.xacro"/>
+    <!-- <xacro:include filename="$(find world_of_stonefish)/world/iceberg.scn.xacro"/> -->
     <xacro:include filename="$(find world_of_stonefish)/vehicles/alpha_rise.scn.xacro"/>
-    <xacro:include filename="$(find world_of_stonefish)/vehicles/wamv.scn.xacro"/>
+    <!-- <xacro:include filename="$(find world_of_stonefish)/vehicles/wamv.scn.xacro"/> -->
     <xacro:alpha_rise robot_name="alpha_rise" xyz="0.0 0.0 0.0" rpy="0.0 0.0 0.0"/>
-    <xacro:wamv robot_name="wamv" xyz="0.0 10.0 0.0" rpy="0.0 0.0 0.0"/>
+    <!-- <xacro:wamv robot_name="wamv" xyz="0.0 10.0 0.0" rpy="0.0 0.0 0.0"/> -->
     <environment>
         <ned latitude="41" longitude="-71"/>

Commit message: rotated the imu orientation of alpha_rise to match the new electronics

File: vehicles/alpha_rise.scn.xacro (robot description, xacro)
@@ -158,5 +158,5 @@
             <sensor name="imu_sf" type="imu" rate="20.0">
                 <link name="Base"/>
-                <origin rpy="0.0 0.0 3.1415926" xyz="-0.65 0.0 -0.05"/>
+                <origin rpy="0.0 0.0 0.0" xyz="-0.65 0.0 -0.05"/>
                 <noise angle="0.0001 0.0001 0.0001" angular_velocity="0.0001" yaw_drift="0.0001" linear_acceleration="0.0001"/>
                 <ros_publisher topic="/${robot_name}/imu/stonefish/data"/>
