Commit message: race and oasis auv config

File: vehicles/alpha_rise.scn.xacro (robot description, xacro)
@@ -24,14 +24,14 @@
                     <material name="Vehicle"/>
                     <look name="yellow"/>
-                    <mass value="38.7"/>
-                    <inertia xyz="1.0 10.0 10.0"/>
+                    <mass value="30.0"/>
+                    <!-- <inertia xyz="1.0 5.0 5.0"/> -->
                     <compound_transform rpy="0.0 0.0 0.0" xyz="0.0 0.0 0.0"/>
-                    <cg xyz="-0.65 0.0 0.1" rpy="0.0 0.0 0.0"/>
+                    <cg xyz="-0.65 0.0 0.00" rpy="0.0 0.0 0.0"/>
                 </external_part>
                 <internal_part name="Foam" type="cylinder" physics="surface" buoyant="true">
-                    <dimensions radius="0.12" height="0.9"/>
+                    <dimensions radius="0.12" height="0.68"/>
                     <origin rpy="0.0 0.0 0.0" xyz="0.0 0.0 0.0"/>
                     <material name="Foam"/>
-                    <mass value="1.5"/>
+                    <mass value="0.1"/>
                     <look name="grey"/>
                     <compound_transform rpy="0.0 1.571 0.0" xyz="-0.65 0.0 -0.1"/>
@@ -92,5 +92,5 @@
                 <link name="Base"/>
                 <origin rpy="0.0 1.571 0.0" xyz="-1.13 0.0 0.0"/>
-                <specs thrust_coeff="0.4472" thrust_coeff_backward="0.3566" torque_coeff="0.01" max_rpm="3000.0"/>
+                <specs thrust_coeff="0.4472" thrust_coeff_backward="0.4472" torque_coeff="0.01" max_rpm="3000.0"/>
                 <propeller diameter="0.08" right="true">
                     <mesh filename="parts/thruster/prop.obj" scale="1.0"/>
@@ -104,5 +104,5 @@
                 <link name="Base"/>
                 <origin rpy="0.0 1.571 0.0" xyz="-0.3545 0.0 0.0"/>
-                <specs thrust_coeff="0.4472" thrust_coeff_backward="0.3566" torque_coeff="0.01" max_rpm="3000.0"/>
+                <specs thrust_coeff="0.4472" thrust_coeff_backward="0.4472" torque_coeff="0.01" max_rpm="3000.0"/>
                 <propeller diameter="0.08" right="true">
                     <mesh filename="parts/thruster/prop.obj" scale="1.0"/>
@@ -194,14 +194,14 @@
                 <ros_publisher topic="/${robot_name}/msis/data"/>
             </sensor> -->
-            <sensor name="MSIS" type="msis">
+            <!-- <sensor name="MSIS" type="msis">
                 <specs step="1" bins="100" horizontal_beam_width="2.0" vertical_beam_width="10.0"/>
                 <settings range_min="0.5" range_max="50.0" rotation_min="-180.0" rotation_max="180.0" gain="1.5"/>
                 <noise multiplicative="0.002" additive="0.003"/>
                 <display colormap="hot"/>
-                <origin xyz="0.0 0.0 0.0" rpy="1.57 0 1.57"/>
+                <origin xyz="0.0 0.0 0.0" rpy="1.57 0 1.57"/> -->
                 <!-- <origin xyz="0.0 0.0 0.0" rpy="1.57 3.14 4.71"/> -->
-                <ros_publisher topic="/${robot_name}/msis/stonefish/data"/>
-                <link name="Base"/>
-            </sensor>
+                <!-- <ros_publisher topic="/${robot_name}/msis/stonefish/data"/>
+                <link name="Base"/>
+            </sensor> -->
             <!-- <sensor name="FLS" type="fls">
                 <specs beams="512" bins="250" horizontal_fov="120.0" vertical_fov="15.0"/>

File: vehicles/race.scn.xacro (robot description, xacro)
@@ -65,5 +65,5 @@
             <actuator name="ThrusterHeaveBow" type="thruster">
                 <link name="Base"/>
-                <origin rpy="0.0 1.571 0.0" xyz="-0.07535 0.0 -0.07535"/>
+                <origin rpy="0.0 -1.571 0.0" xyz="-0.07535 0.0 -0.07535"/>
                 <specs thrust_coeff="0.4472" thrust_coeff_backward="0.3566" torque_coeff="0.01" max_rpm="3000.0"/>
                 <propeller diameter="0.08" right="true">
@@ -76,5 +76,5 @@
             <actuator name="ThrusterHeaveSternPort" type="thruster">
                 <link name="Base"/>
-                <origin rpy="0.0 1.571 0.0" xyz="-0.56 -0.1034 -0.07535"/>
+                <origin rpy="0.0 -1.571 0.0" xyz="-0.56 -0.1034 -0.07535"/>
                 <specs thrust_coeff="0.4472" thrust_coeff_backward="0.3566" torque_coeff="0.01" max_rpm="3000.0"/>
                 <propeller diameter="0.08" right="true">
@@ -87,5 +87,5 @@
             <actuator name="ThrusterHeaveSternStbd" type="thruster">
                 <link name="Base"/>
-                <origin rpy="0.0 1.571 0.0" xyz="-0.56 0.1034 -0.07535"/>
+                <origin rpy="0.0 -1.571 0.0" xyz="-0.56 0.1034 -0.07535"/>
                 <specs thrust_coeff="0.4472" thrust_coeff_backward="0.3566" torque_coeff="0.01" max_rpm="3000.0"/>
                 <propeller diameter="0.08" right="true">
@@ -144,16 +144,16 @@
                 <ros_publisher topic="/${robot_name}/gps/fix"/>
             </sensor>
-            <sensor name="Cam" rate="5.0" type="camera">
+            <!-- <sensor name="Cam" rate="5.0" type="camera">
                 <link name="Base"/>
                 <specs resolution_x="800" resolution_y="600" horizontal_fov="60.0"/>
                 <origin xyz="0.0 0.0 -0.05" rpy="1.571 0.0 1.571"/>
                 <ros_publisher topic="/${robot_name}/camera/data"/>
-            </sensor>
-            <light name="Spot">
+            </sensor> -->
+            <!-- <light name="Spot">
                 <link name="Base"/>
                 <specs radius="0.01" cone_angle="120.0" illuminance="20000.0"/>
                 <color temperature="5600.0"/>
                 <origin xyz="0.0 0.0 -0.1" rpy="0.0 1.571 0.0"/>
-            </light>
+            </light> -->
             <world_transform rpy="${rpy}" xyz="${xyz}"/>
             <!-- <world_transform xyz="0.0 0.0 0.0" rpy="0.0 0.0 0.0"/> -->

File: world/ocean.scn.xacro (robot description, xacro)
@@ -32,9 +32,9 @@
     <static name="Bottom" type="model">
         <physical>
-            <mesh filename="objects/flat_terrain.obj" scale="2.0" convex="true"/>
+            <mesh filename="objects/flat_terrain.obj" scale="10.0" convex="true"/>
             <origin xyz="0.0 0.0 0.0" rpy="0.0 0.0 0.0"/>
         </physical>
         <visual>
-            <mesh filename="objects/flat_terrain.obj" scale="2.0"/>
+            <mesh filename="objects/flat_terrain.obj" scale="10.0"/>
             <origin xyz="0.0 0.0 0.0" rpy="0.0 0.0 0.0"/>
         </visual>
