Commit message: added a cage

File: vehicles/race.scn.xacro (robot description, xacro)
@@ -25,13 +25,13 @@
                     <look name="yellow"/>
                     <mass value="25.0"/>
-                    <inertia xyz="1.0 10.0 10.0"/>
+                    <!-- <inertia xyz="1.0 10.0 10.0"/> -->
                     <compound_transform rpy="0.0 0.0 0.0" xyz="0.0 0.0 0.0"/>
                     <cg xyz="-0.456 0.0 0.0" rpy="0.0 0.0 0.0"/>
                 </external_part>
                 <internal_part name="Foam" type="box" physics="surface" buoyant="true">
-                    <dimensions xyz="0.8 0.25 0.15"/>
+                    <dimensions xyz="0.8 0.21 0.15"/>
                     <origin rpy="0.0 0.0 0.0" xyz="-0.456 0.0 -0.1"/>
                     <material name="Foam"/>
-                    <mass value="0.1"/>
+                    <mass value="0.15"/>
                     <look name="grey"/>
                     <compound_transform rpy="0.0 0.0 0.0" xyz="0.0 0.0 0.0"/>
@@ -144,4 +144,16 @@
                 <ros_publisher topic="/${robot_name}/gps/fix"/>
             </sensor>
+            <sensor name="Cam" rate="5.0" type="camera">
+                <link name="Base"/>
+                <specs resolution_x="800" resolution_y="600" horizontal_fov="60.0"/>
+                <origin xyz="0.0 0.0 -0.05" rpy="1.571 0.0 1.571"/>
+                <ros_publisher topic="/${robot_name}/camera/data"/>
+            </sensor>
+            <light name="Spot">
+                <link name="Base"/>
+                <specs radius="0.01" cone_angle="120.0" illuminance="20000.0"/>
+                <color temperature="5600.0"/>
+                <origin xyz="0.0 0.0 -0.1" rpy="0.0 1.571 0.0"/>
+            </light>
             <world_transform rpy="${rpy}" xyz="${xyz}"/>
             <!-- <world_transform xyz="0.0 0.0 0.0" rpy="0.0 0.0 0.0"/> -->

File: world/ocean_race.scn.xacro (robot description, xacro)
@@ -43,3 +43,17 @@
         <world_transform xyz="0.0 0.0 40.0" rpy="0.0 0.0 0.0"/>
     </static>
+    <static name="cage" type="model">
+        <physical>
+            <mesh filename="objects/cage.obj" scale="0.001" convex="false"/>
+            <origin xyz="0 0 0.0" rpy="0.0 0.0 0.0"/>
+        </physical>
+        <visual>
+            <mesh filename="objects/cage.obj" scale="0.001"/>
+            <origin xyz="0 0 0.0" rpy="0.0 0.0 0.0"/>
+        </visual>
+        <material name="Aluminium"/>
+        <look name="black"/>
+        <cg xyz=" 0.0 0 0.0" rpy="0.0 0.0 0.0"/>
+        <world_transform xyz="6.0 0.0 2" rpy="3.1415926 0.0 0.0"/>
+    </static>
 </scenario>

Commit message: rotated the race auv surge thruster for testing

File: vehicles/race.scn.xacro (robot description, xacro)
@@ -98,5 +98,5 @@
             <actuator name="ThrusterSurgePort" type="thruster">
                 <link name="Base"/>
-                <origin rpy="0.0 0.0 -0.52" xyz="-0.86 -0.125 -0.05485"/>
+                <origin rpy="0.0 0.8 -0.52" xyz="-0.86 -0.125 -0.05485"/>
                 <specs thrust_coeff="0.4472" thrust_coeff_backward="0.3566" torque_coeff="0.01" max_rpm="3000.0"/>
                 <propeller diameter="0.08" right="true">
@@ -109,5 +109,5 @@
             <actuator name="ThrusterSurgeStbd" type="thruster">
                 <link name="Base"/>
-                <origin rpy="0.0 0.0 0.52" xyz="-0.86 0.125 -0.05485"/>
+                <origin rpy="0.0 0.8 0.52" xyz="-0.86 0.125 -0.05485"/>
                 <specs thrust_coeff="0.4472" thrust_coeff_backward="0.3566" torque_coeff="0.01" max_rpm="3000.0"/>
                 <propeller diameter="0.08" right="true">
