Commit message: stonefish setup for alpha_img_auv

File: vehicles/alpha_img.scn.xacro (robot description, xacro)
@@ -12,12 +12,15 @@
     <xacro:macro name="alpha_img" params="xyz rpy robot_name">
         <robot name="${robot_name}" fixed="false" self_collisions="false">
+            <!-- ==================================================================== -->
+            <!--                             Vehicle Base                             -->
+            <!-- ==================================================================== -->
             <base_link name="Vehicle" type="compound" physics="submerged">
                 <external_part name="Hull" type="model" physics="submerged" buoyant="false">
                     <physical>
-                        <mesh filename="parts/body/hull_mk2_reduced.obj" scale="0.001"/>
+                        <mesh filename="parts/body/alpha_img_auv.obj" scale="0.001"/>
                         <origin rpy="1.5707 0.0 0.0" xyz="0.0 0.0 0.0"/>
                     </physical>
                     <visual>
-                        <mesh filename="parts/body/hull_mk2_visual.obj" scale="0.001"/>
+                        <mesh filename="parts/body/alpha_img_auv.obj" scale="0.001"/>
                         <origin rpy="1.5707 0.0 0.0" xyz="0.0 0.0 0.0"/>
                     </visual>
@@ -53,9 +56,9 @@
                     <physical>
                         <mesh filename="parts/thruster/duct.obj" scale="0.0015"/>
-                        <origin rpy="0.0 1.571 0.0" xyz="-1.5 0.0 0.0"/>
+                        <origin rpy="0.0 1.571 0.0" xyz="-1.4 0.0 0.0"/>
                     </physical>
                     <visual>
                         <mesh filename="parts/thruster/duct.obj" scale="0.0015"/>
-                        <origin rpy="0.0 1.571 0.0" xyz="-1.5 0.0 0.0"/>
+                        <origin rpy="0.0 1.571 0.0" xyz="-1.4 0.0 0.0"/>
                     </visual>
                     <material name="Neutral"/>
@@ -64,6 +67,10 @@
                 </external_part>
             </base_link>
-            <!-- the actual base frame  -->
-            <link name="Base" type="box" physics="submerged">
+            <!-- ==================================================================== -->
+            <!--                           Adjusted Frames                            -->
+            <!-- ==================================================================== -->
+            <!-- CAD_link: which is the original point of a obj file,
+                 it may difference from the vehicle nose  -->
+            <link name="CAD_link" type="box" physics="submerged">
                 <dimensions xyz="0.01 0.02 0.01"/>
                 <origin xyz="0.0 0.0 0.0" rpy="0.0 0.0 0.0"/>
@@ -71,14 +78,57 @@
                 <look name="Green"/>
             </link>
-            <joint name="Joint1" type="fixed">
+            <joint name="Joint_CAD" type="fixed">
                 <parent name="Vehicle"/>
-                <child name="Base"/>
+                <child name="CAD_link"/>
                 <origin xyz="0.0 0.0 0.0" rpy="0.0 0.0 0.0"/>
                 <axis xyz="1.0 0.0 0.0"/>
             </joint>
-            <!--  -->
+            <!-- Nose_link: the frame located on vehicle nose, used to measurement relative
+                 position between sensor and nose in a CAD model (obj file) -->
+            <link name="Nose_link" type="box" physics="submerged">
+                <dimensions xyz="0.01 0.02 0.01"/>
+                <origin xyz="0.0 0.0 0.0" rpy="0.0 0.0 0.0"/>
+                <material name="Neutral"/>
+                <look name="Green"/>
+            </link>
+            <joint name="Joint_Nose" type="fixed">
+                <parent name="CAD_link"/>
+                <child name="Nose_link"/>
+                <origin xyz="0.0 0.0 0.0" rpy="0.0 0.0 0.0"/>
+                <axis xyz="1.0 0.0 0.0"/>
+            </joint>
+            <!-- ==================================================================== -->
+            <!--                         All the thrusters                            -->
+            <!-- ==================================================================== -->
+            <!-- Vetrical Front Thruster -->
+            <actuator name="ThrusterHeaveBow" type="thruster">
+                <link name="Nose_link"/>
+                <origin rpy="0.0 1.571 0.0" xyz="-0.2295 0.0 0.0"/>
+                <specs thrust_coeff="0.4472" thrust_coeff_backward="0.3566" torque_coeff="0.01" max_rpm="3000.0"/>
+                <propeller diameter="0.08" right="true">
+                    <mesh filename="parts/thruster/prop.obj" scale="1.0"/>
+                    <mesh filename="prop.obj" scale="1.0"/>
+                    <material name="Neutral"/>
+                    <look name="white"/>
+                </propeller>
+                <ros_subscriber topic="/${robot_name}/control/thruster/heave_bow"/>
+            </actuator>
+            <!-- Vetrical Back Thruster -->
+            <actuator name="ThrusterHeaveStern" type="thruster">
+                <link name="Nose_link"/>
+                <origin rpy="0.0 1.571 0.0" xyz="-0.88 0.0 0.0"/>
+                <specs thrust_coeff="0.4472" thrust_coeff_backward="0.3566" torque_coeff="0.01" max_rpm="3000.0"/>
+                <propeller diameter="0.08" right="true">
+                    <mesh filename="parts/thruster/prop.obj" scale="1.0"/>
+                    <mesh filename="prop.obj" scale="1.0"/>
+                    <material name="Neutral"/>
+                    <look name="white"/>
+                </propeller>
+                <ros_subscriber topic="/${robot_name}/control/thruster/heave_stern"/>
+            </actuator>
+            <!-- -->
             <actuator name="ThrusterSwayBow" type="thruster">
-                <link name="Base"/>
-                <origin rpy="0.0 0.0 -1.5707963" xyz="-0.2295 0.0 0.0"/>
+                <link name="Nose_link"/>
+                <origin rpy="0.0 0.0 -1.5707963" xyz="-1.005 0.0 0.0"/>
                 <specs thrust_coeff="0.4472" thrust_coeff_backward="0.3566" torque_coeff="0.01" max_rpm="3000.0"/>
                 <propeller diameter="0.08" right="true">
@@ -89,31 +139,8 @@
                 <ros_subscriber topic="/${robot_name}/control/thruster/sway_bow"/>
             </actuator>
-            <actuator name="ThrusterHeaveStern" type="thruster">
-                <link name="Base"/>
-                <origin rpy="0.0 1.571 0.0" xyz="-1.13 0.0 0.0"/>
-                <specs thrust_coeff="0.4472" thrust_coeff_backward="0.3566" torque_coeff="0.01" max_rpm="3000.0"/>
-                <propeller diameter="0.08" right="true">
-                    <mesh filename="parts/thruster/prop.obj" scale="1.0"/>
-                    <mesh filename="prop.obj" scale="1.0"/>
-                    <material name="Neutral"/>
-                    <look name="white"/>
-                </propeller>
-                <ros_subscriber topic="/${robot_name}/control/thruster/heave_stern"/>
-            </actuator>
-            <actuator name="ThrusterHeaveBow" type="thruster">
-                <link name="Base"/>
-                <origin rpy="0.0 1.571 0.0" xyz="-0.3545 0.0 0.0"/>
-                <specs thrust_coeff="0.4472" thrust_coeff_backward="0.3566" torque_coeff="0.01" max_rpm="3000.0"/>
-                <propeller diameter="0.08" right="true">
-                    <mesh filename="parts/thruster/prop.obj" scale="1.0"/>
-                    <mesh filename="prop.obj" scale="1.0"/>
-                    <material name="Neutral"/>
-                    <look name="white"/>
-                </propeller>
-                <ros_subscriber topic="/${robot_name}/control/thruster/heave_bow"/>
-            </actuator>
+            <!-- -->
             <actuator name="ThrusterSurge" type="thruster">
-                <link name="Base"/>
-                <origin rpy="0.0 0.0 0.0" xyz="-1.5 0.0 0.0"/>
+                <link name="Nose_link"/>
+                <origin rpy="0.0 0.0 0.0" xyz="-1.4 0.0 0.0"/>
                 <specs thrust_coeff="1.7568" thrust_coeff_backward="1.0882" torque_coeff="0.01" max_rpm="3000.0"/>
                 <propeller diameter="0.08" right="true">
@@ -126,29 +153,18 @@
                 <ros_subscriber topic="/${robot_name}/control/thruster/surge"/>
             </actuator>
-<!--
-            <actuator name="Rudder" type="rudder">
-                <link name="Base"/> -->
-            <!-- <actuator name="Rudder" type="rudder">
-                <link name="Base"/> -->
-                <!-- a manual angle -->
-                <!-- <origin rpy="0.0 0.0 0.2" xyz="0.0 0.0 0.0"/>  -->
-                <!-- <origin rpy="0.0 0.0 0.0" xyz="0.0 0.0 0.0"/>
-                <specs drag_coeff="1.0" lift_coeff="3.0" max_angle="0.6" inverted="false" area="0.06"/>
-                <visual>
-                    <mesh filename="parts/others/rudder.obj" scale="0.002"/>
-                    <material name="Neutral"/>
-                    <look name="black"/>
-                    <origin rpy="-1.571 1.571 0.3" xyz="-1.2 0.0 0.2"/>
-                </visual>
-            </actuator> -->
+            <!-- ==================================================================== -->
+            <!--                          Navigation Sensors                          -->
+            <!-- ==================================================================== -->
+            <!-- -->
             <sensor name="pressure" type="pressure" rate="5.0">
-                <link name="Base"/>
-                <origin rpy="0.0 0.0 0.0" xyz="-1.20 0.0 0.0"/>
+                <link name="Nose_link"/>
+                <origin rpy="0.0 0.0 0.0" xyz="-0.4073 0.0625 0.0"/>
                 <noise pressure="2.0"/>
                 <ros_publisher topic="/${robot_name}/pressure"/>
             </sensor>
+            <!-- -->
             <sensor name="dvl_sf" type="dvl" rate="5.0">
-                <link name="Base"/>
-                <origin rpy="3.1415926 0.0 0.0" xyz="-0.65 0.0 0.1"/>
+                <link name="Nose_link"/>
+                <origin rpy="3.1415926 0.0 0.0" xyz="-1.005 0.0 0.1"/>
                 <specs beam_angle="30.0"/>
                 <range velocity="9.0 9.0 9.0" altitude_min="0.2" altitude_max="200.0"/>
@@ -156,12 +172,13 @@
                 <ros_publisher topic="/${robot_name}/dvl/twist" altitude_topic="/${robot_name}/dvl/altitude"/>
             </sensor>
+            <!-- -->
             <sensor name="imu_sf" type="imu" rate="20.0">
-                <link name="Base"/>
-                <origin rpy="0.0 0.0 0.0" xyz="-0.65 0.0 -0.05"/>
+                <link name="Nose_link"/>
+                <origin rpy="0.0 0.0 0.0" xyz="-0.6867 0.0625 0.0381"/>
                 <noise angle="0.0001 0.0001 0.0001" angular_velocity="0.0001" yaw_drift="0.0001" linear_acceleration="0.0001"/>
                 <ros_publisher topic="/${robot_name}/imu/stonefish/data"/>
             </sensor>
             <sensor name="gps" type="gps" rate="1.0">
-                <link name="Base"/>
+                <link name="Nose_link"/>
                 <origin rpy="0.0 0.0 0.0" xyz="-0.7 0.0 -0.3"/>
                 <noise ned_position="0.0"/>
@@ -172,26 +189,11 @@
                 <history samples="1"/>
                 <origin xyz="0.0 0.0 0.0" rpy="3.1415926 0.0 -1.5707963"/>
-                <link name="Base"/>
+                <link name="Nose_link"/>
                 <ros_publisher topic="/${robot_name}/sf/odometry"/>
             </sensor> -->
-            <!-- perception sensors -->
-            <!-- <sensor name="mss" rate="5.0" type="profiler">
-                <specs fov="90.0" steps="100"/>
-                <range distance_min="0.5" distance_max="100.0"/>
-                <noise distance="0.05"/>
-                <history samples="1"/>
-                <origin xyz="0.0 0.0 0.0" rpy="0.0 -1.5707963 0.0"/>
-                <link name="Base"/>
-                <ros_publisher topic="/${robot_name}/MSS/data"/>
-            </sensor> -->
-            <!-- <sensor name="msis" type="msis">
-                <specs step="1.8" bins="1250" horizontal_beam_width="1.5" vertical_beam_width="15.0"/>
-                <settings range_min="0.75" range_max="50.0" rotation_min="-45.0" rotation_max="45.0" gain="3.5"/>
-                <noise multiplicative="0.02" additive="0.03"/>
-                <display colormap="hot"/>
-                <origin xyz="0.0 0.0 0.0" rpy="0.0 0.0 1.5707963"/>
-                <link name="Base"/>
-                <ros_publisher topic="/${robot_name}/msis/data"/>
-            </sensor> -->
+            <!-- ==================================================================== -->
+            <!--                          Perception Sensors                          -->
+            <!-- ==================================================================== -->
+            <!-- -->
             <sensor name="MSIS" type="msis">
                 <specs step="1" bins="100" horizontal_beam_width="2.0" vertical_beam_width="10.0"/>
@@ -199,20 +201,29 @@
                 <noise multiplicative="0.002" additive="0.003"/>
                 <display colormap="hot"/>
-                <origin xyz="0.0 0.0 0.0" rpy="1.57 0 1.57"/>
-                <!-- <origin xyz="0.0 0.0 0.0" rpy="1.57 3.14 4.71"/> -->
+                <origin xyz="-0.01 -0.12192 0.0" rpy="3.1415926 0 3.1415926"/>
                 <ros_publisher topic="/${robot_name}/msis/stonefish/data"/>
-                <link name="Base"/>
-            </sensor>
-            <!-- <sensor name="FLS" type="fls">
-                <specs beams="512" bins="250" horizontal_fov="120.0" vertical_fov="15.0"/>
-                <settings range_min="0.5" range_max="100.0" gain="1.5"/>
+                <link name="Nose_link"/>
+            </sensor>
+            <!-- Simulated M750d 750kHz -->
+            <sensor name="FLS" type="fls">
+                <specs beams="512" bins="667" horizontal_fov="130.0" vertical_fov="20.0"/>
+                <settings range_min="0.1" range_max="40.0" gain="1.5"/>
                 <noise multiplicative="0.01" additive="0.02"/>
                 <display colormap="hot"/>
-                <origin xyz="0.0 0.0 0.0" rpy="1.5707963 0.0 1.5707963"/>
-                <link name="Base"/>
+                <origin xyz="0.0 0.04 0.09" rpy="1.3107963 0 1.5707963"/>
+                <link name="Nose_link"/>
+                <ros_publisher topic="/${robot_name}/FLS/data"/>
+            </sensor>
+            <!-- Simulated M750d 1.2MHz -->
+            <!-- <sensor name="FLS" type="fls">
+                <specs beams="512" bins="667" horizontal_fov="70.0" vertical_fov="12.0"/>
+                <settings range_min="0.1" range_max="40.0" gain="1.5"/>
+                <noise multiplicative="0.01" additive="0.02"/>
+                <display colormap="hot"/>
+                <origin xyz="0.0 0.04 0.09" rpy="1.3107963 0 1.5707963"/>
+                <link name="Nose_link"/>
                 <ros_publisher topic="/${robot_name}/FLS/data"/>
             </sensor> -->
             <world_transform rpy="${rpy}" xyz="${xyz}"/>
-            <!-- <world_transform xyz="0.0 0.0 0.0" rpy="0.0 0.0 0.0"/> -->
         </robot>
     </xacro:macro>

File: world/tank_img.scn.xacro (robot description, xacro)
@@ -8,4 +8,7 @@
 -->
 <scenario xmlns:xacro="http://ros.org/wiki/xacro">
+    <!-- <xacro:arg name="robot_name" default="changeme"/> -->
+    <!-- <xacro:include filename="$(find world_of_stonefish)/vehicles/alpha_std.scn.xacro"/> -->
+    <!-- <xacro:alpha_std robot_name="$(arg robot_name)" xyz="0.0 0.0 0.0" rpy="0.0 0.0 0.0"/> -->
     <xacro:arg name="robot_name" default="changeme"/>
     <xacro:include filename="$(find world_of_stonefish)/vehicles/$(arg robot_name).scn.xacro"/>
@@ -14,15 +17,10 @@
         <ned latitude="41" longitude="-71"/>
         <ocean>
-            <water density="1031.0" jerlov="0.2"/>
-            <!-- <waves height="0.0"/> -->
+            <water density="1000.0" jerlov="0.2"/>
+            <waves height="0.0"/>
             <particles enabled="true"/>
             <current type="uniform">
                 <velocity xyz="0.0 0.0 0.0"/>
             </current>
-            <!-- <current type="jet">
-                <center xyz="0.0 0.0 3.0"/>
-                <outlet radius="0.2"/>
-                <velocity xyz="0.0 2.0 0.0"/>
-            </current> -->
         </ocean>
         <atmosphere>
@@ -30,16 +28,16 @@
         </atmosphere>
     </environment>
-    <static name="Bottom" type="model">
+    <static name="tank" type="model">
         <physical>
-            <mesh filename="objects/flat_terrain.obj" scale="2.0" convex="true"/>
+            <mesh filename="objects/tank.obj" scale="1.0" convex="false"/>
             <origin xyz="0.0 0.0 0.0" rpy="0.0 0.0 0.0"/>
         </physical>
         <visual>
-            <mesh filename="objects/flat_terrain.obj" scale="2.0"/>
+            <mesh filename="objects/tank.obj" scale="1.0"/>
             <origin xyz="0.0 0.0 0.0" rpy="0.0 0.0 0.0"/>
         </visual>
         <material name="Rock"/>
         <look name="Gray"/>
-        <world_transform xyz="0.0 0.0 40.0" rpy="0.0 0.0 0.0"/>
+        <world_transform xyz="0.0 0.0 18.0" rpy="3.1415926 0.0 0.0"/>
     </static>
 </scenario>

Commit message: update alpha_img

File: vehicles/alpha_img.scn.xacro (robot description, xacro)
@@ -185,11 +185,12 @@
                 <ros_publisher topic="/${robot_name}/gps/fix"/>
             </sensor>
-            <!-- <sensor name="odom" rate="10.0" type="odometry">
-                <noise position="0.00" velocity="0.00" angle="0.0" angular_velocity="0.00"/>
+            <!-- Odometry: Groundtruth on IMU frame -->
+            <sensor name="Odometry" rate="10.0" type="odometry">
+                <noise position="0.0" velocity="0.0" angle="0.0" angular_velocity="0.0"/>
                 <history samples="1"/>
-                <origin xyz="0.0 0.0 0.0" rpy="3.1415926 0.0 -1.5707963"/>
-                <link name="Nose_link"/>
+                <link name="Nose_link"/>
+                <origin rpy="0.0 0.0 0.0" xyz="-0.6867 0.0625 0.0381"/>
                 <ros_publisher topic="/${robot_name}/sf/odometry"/>
-            </sensor> -->
+            </sensor>
             <!-- ==================================================================== -->
             <!--                          Perception Sensors                          -->
