Commit message: Race2 Starboard scn

File: vehicles/race2.scn.xacro (robot description, xacro)
@@ -2,6 +2,6 @@
 <!--
     This file is part of RACE AUV project.
-    Author: Farhang Naderi,Ming
-    Email: farhang.nba@gmail.com,farhang.naderi@uri.edu
+    Author: Farhang Naderi,Mingxi Zhou
+    Email: farhang.nba@gmail.com,farhang.naderi@uri.edu,mzhou@uri.edu
     Year: 2023
     Copyright (C) 2023 Smart Ocean Systems Laboratory
@@ -200,12 +200,12 @@
             <joint name="surge_starboard_servo_joint" type="fixed">
                 <parent name="Vehicle"/>
-                <child name="surge_port_servo_link"/>
-                <origin rpy="-1.571 0.0 -0.52" xyz="-0.86 0.125 -0.05485"/>
+                <child name="surge_starboard_servo_link"/>
+                <origin rpy="1.571 0.0 0.52" xyz="-0.86 0.125 -0.05485"/>
                 <axis xyz="1.0 0.0 0.0"/>
             </joint>
                  <!-- revolute joint from servo to duct -->
             <joint name="surge_starboard_servo2duct_joint" type="revolute">
-                <parent name="surge_port_servo_link"/>
-                <child name="surge_port_duct_link"/>
+                <parent name="surge_starboard_servo_link"/>
+                <child name="surge_starboard_duct_link"/>
                 <origin rpy="0.0 0.0 0.0" xyz="0.0 0.0 0.0"/>
                 <axis xyz="0.0 0.0 1.0"/>
@@ -214,6 +214,6 @@
                 <!-- fixed joint between thruster and duct -->
             <joint name="surge_starboard_thruster_joint" type="fixed">
-                <parent name="surge_port_duct_link"/>
-                <child name="surge_port_thruster_link"/>
+                <parent name="surge_starboard_duct_link"/>
+                <child name="surge_starboard_thruster_link"/>
                 <origin rpy="0.0 0.0 0.0" xyz="0.0 0.0 0.0"/>
                 <axis xyz="1.0 0.0 0.0"/>
@@ -221,5 +221,5 @@
                 <!-- attached servo to the joint between servo and duct  -->
             <actuator name="surge_starboard_servo" type="servo">
-                <joint name="surge_port_servo2duct_joint"/>
+                <joint name="surge_starboard_servo2duct_joint"/>
                 <controller position_gain="1.1" velocity_gain="0.1" max_torque="10.0"/>
             </actuator>
@@ -236,42 +236,4 @@
                 <ros_subscriber topic="/${robot_name}/control/thruster/surge_starboard"/>
             </actuator>
-            <!-- <link name="surge_starboard_duct_link" type="compound" physics="submerged">
-                <external_part name="SurgeStarboardDuct" type="model" physics="submerged" buoyant="true">
-                    <physical>
-                        <mesh filename="parts/thruster/duct_reduced.obj" scale="0.001"/>
-                        <origin rpy="0.0 0.0 0.0" xyz="0.0 0.0 0.0"/>
-                    </physical>
-                    <visual>
-                        <mesh filename="parts/thruster/duct.obj" scale="0.001"/>
-                        <origin rpy="0.0 0.0 0.0" xyz="0.0 0.0 0.0"/>
-                    </visual>
-                    <material name="Neutral"/>
-                    <look name="black"/>
-                    <compound_transform rpy="0.0 -1.57 0.0" xyz="0.0 0.0 0.0"/>
-                </external_part>
-            </link>
-            <actuator name="ThrusterSurgeStbd" type="thruster">
-                <link name="surge_starboard_base_link"/>
-                <origin rpy="0.0 0.0 0.0" xyz="0.0 0.0 0.0"/>
-                <specs thrust_coeff="0.4472" thrust_coeff_backward="0.3566" torque_coeff="0.01" max_rpm="3000.0"/>
-                <propeller diameter="0.08" right="true">
-                    <mesh filename="parts/thruster/prop.obj" scale="1.0"/>
-                    <material name="Neutral"/>
-                    <look name="white"/>
-                </propeller>
-                <ros_subscriber topic="/${robot_name}/control/thruster/surge_starboard"/>
-            </actuator>
-            <joint name="surge_starboard_servo_joint" type="revolute">
-                <parent name="Vehicle"/>
-                <child name="surge_starboard_duct_link"/>
-                <origin rpy="0.0 0.0 0.52" xyz="-0.86 0.125 -0.05485"/>
-                <axis xyz="0.0 1.0 0.0"/>
-                <limits min="-1.571" max="1.571"/>
-            </joint>
-            <actuator name="ServoSurgeStarboard" type="servo">
-                <joint name="surge_starboard_servo_joint"/>
-                <controller position_gain="1.1" velocity_gain="0.1" max_torque="10.0"/>
-            </actuator> -->
-            <!-- <ros_joint_subscriber joint_name="surge_starboard_servo_joint" topic="/${robot_name}/joint/servo/starboard" control_mode="position" /> -->
             <!-- End: Starboard Surge -->
             <sensor name="pressure" type="pressure" rate="5.0">

Commit message: race2 scn

File: vehicles/race2.scn.xacro (robot description, xacro)
@@ -74,5 +74,5 @@
                 <ros_subscriber topic="/${robot_name}/control/thruster/heave_bow"/>
             </actuator>
-            <actuator name="ThrusterHeaveSternPort" type="thruster">
+            <!-- <actuator name="ThrusterHeaveSternPort" type="thruster">
                 <link name="Base"/>
                 <origin rpy="0.0 -1.571 0.0" xyz="-0.56 -0.1034 -0.07535"/>
@@ -95,5 +95,5 @@
                 </propeller>
                 <ros_subscriber topic="/${robot_name}/control/thruster/heave_stern_stbd"/>
-            </actuator>
+            </actuator> -->
             <!-- Start: Port Surge -->
             <!-- servo link -->
@@ -131,5 +131,5 @@
                 <parent name="Vehicle"/>
                 <child name="surge_port_servo_link"/>
-                <origin rpy="-1.571 0.0 -0.52" xyz="-0.86 -0.125 -0.05485"/>
+                <origin rpy="1.571 0.0 -0.52" xyz="-0.86 -0.125 -0.05485"/>
                 <axis xyz="1.0 0.0 0.0"/>
             </joint>
@@ -152,5 +152,5 @@
             <actuator name="surge_port_servo" type="servo">
                 <joint name="surge_port_servo2duct_joint"/>
-                <controller position_gain="1.1" velocity_gain="0.1" max_torque="10.0"/>
+                <controller position_gain="0.03" velocity_gain="1.0" max_torque="0.2"/>
             </actuator>
                 <!-- attach thruster/propeller at the thruster link -->
@@ -201,5 +201,5 @@
                 <parent name="Vehicle"/>
                 <child name="surge_starboard_servo_link"/>
-                <origin rpy="1.571 0.0 0.52" xyz="-0.86 0.125 -0.05485"/>
+                <origin rpy="-1.571 0.0 0.52" xyz="-0.86 0.125 -0.05485"/>
                 <axis xyz="1.0 0.0 0.0"/>
             </joint>
@@ -222,5 +222,5 @@
             <actuator name="surge_starboard_servo" type="servo">
                 <joint name="surge_starboard_servo2duct_joint"/>
-                <controller position_gain="1.1" velocity_gain="0.1" max_torque="10.0"/>
+                <controller position_gain="0.03" velocity_gain="1.0" max_torque="0.2"/>
             </actuator>
                 <!-- attach thruster/propeller at the thruster link -->

Commit message: servo linke placement updated based on hardware

File: vehicles/race2.scn.xacro (robot description, xacro)
@@ -131,5 +131,5 @@
                 <parent name="Vehicle"/>
                 <child name="surge_port_servo_link"/>
-                <origin rpy="1.571 0.0 -0.52" xyz="-0.86 -0.125 -0.05485"/>
+                <origin rpy="1.571 1.78 -0.52" xyz="-0.86 -0.125 -0.05485"/>
                 <axis xyz="1.0 0.0 0.0"/>
             </joint>
@@ -201,5 +201,5 @@
                 <parent name="Vehicle"/>
                 <child name="surge_starboard_servo_link"/>
-                <origin rpy="-1.571 0.0 0.52" xyz="-0.86 0.125 -0.05485"/>
+                <origin rpy="-1.571 -1.78 0.52" xyz="-0.86 0.125 -0.05485"/>
                 <axis xyz="1.0 0.0 0.0"/>
             </joint>

Commit message: Vehicle update for ROVMaker servo (#13)
* Vehicle update for ROVMaker servo

* servo linke placement updated based on hardware

File: vehicles/race2.scn.xacro (robot description, xacro)
@@ -131,5 +131,5 @@
                 <parent name="Vehicle"/>
                 <child name="surge_port_servo_link"/>
-                <origin rpy="1.571 0.0 -0.52" xyz="-0.86 -0.125 -0.05485"/>
+                <origin rpy="1.571 1.78 -0.52" xyz="-0.86 -0.125 -0.05485"/>
                 <axis xyz="1.0 0.0 0.0"/>
             </joint>
@@ -140,5 +140,5 @@
                 <origin rpy="0.0 0.0 0.0" xyz="0.0 0.0 0.0"/>
                 <axis xyz="0.0 0.0 1.0"/>
-                <limits min="-1.571" max="1.571"/>
+                <limits min="-3.14" max="3.14"/>
             </joint>
                 <!-- fixed joint between thruster and duct -->
@@ -201,5 +201,5 @@
                 <parent name="Vehicle"/>
                 <child name="surge_starboard_servo_link"/>
-                <origin rpy="-1.571 0.0 0.52" xyz="-0.86 0.125 -0.05485"/>
+                <origin rpy="-1.571 -1.78 0.52" xyz="-0.86 0.125 -0.05485"/>
                 <axis xyz="1.0 0.0 0.0"/>
             </joint>
@@ -210,5 +210,5 @@
                 <origin rpy="0.0 0.0 0.0" xyz="0.0 0.0 0.0"/>
                 <axis xyz="0.0 0.0 1.0"/>
-                <limits min="-1.571" max="1.571"/>
+                <limits min="-3.14" max="3.14"/>
             </joint>
                 <!-- fixed joint between thruster and duct -->

Commit message: race 2 physics and limits change

File: vehicles/race2.scn.xacro (robot description, xacro)
@@ -25,11 +25,12 @@
                     <look name="yellow"/>
                     <mass value="25.0"/>
-                    <!-- <inertia xyz="1.0 10.0 10.0"/> -->
-                    <compound_transform rpy="0.0 0.0 0.0" xyz="0.0 0.0 0.0"/>
-                    <cg xyz="-0.456 0.0 0.0" rpy="0.0 0.0 0.0"/>
+                    <!-- disable for stonefish to determine it -->
+                    <!-- <inertia xyz="5.0 10.0 10.0"/>  -->
+                    <compound_transform rpy="0.0 0.0 0.0" xyz="0.0 0.0 0.0"/>
+                    <cg xyz="-0.456 0.0 -0.1" rpy="0.0 0.0 0.0"/>
                 </external_part>
                 <internal_part name="Foam" type="box" physics="surface" buoyant="true">
                     <dimensions xyz="0.8 0.21 0.15"/>
-                    <origin rpy="0.0 0.0 0.0" xyz="-0.456 0.0 -0.1"/>
+                    <origin rpy="0.0 0.0 0.0" xyz="-0.456 0.0 -0.2"/>
                     <material name="Foam"/>
                     <mass value="0.15"/>
@@ -45,4 +46,16 @@
                 <look name="Green"/>
             </link>
+            <!-- <link name="Base2" type="box" physics="submerged">
+                <dimensions xyz="0.01 0.02 0.01"/>
+                <origin xyz="0.0 0.0 0.0" rpy="0.0 0.0 0.0"/>
+                <material name="Neutral"/>
+                <look name="Green"/>
+            </link>
+            <joint name="Joint1" type="fixed">
+                <parent name="Base"/>
+                <child name="Base2"/>
+                <origin xyz="0.2 0.0 0.0" rpy="0.0 0.0 0.0"/>
+                <axis xyz="1.0 0.0 0.0"/>
+            </joint> -->
             <joint name="Joint1" type="fixed">
                 <parent name="Vehicle"/>
@@ -131,5 +144,6 @@
                 <parent name="Vehicle"/>
                 <child name="surge_port_servo_link"/>
-                <origin rpy="1.571 1.78 -0.52" xyz="-0.86 -0.125 -0.05485"/>
+                <!-- <origin rpy="1.571 1.78 -0.52" xyz="-0.86 -0.125 -0.05485"/> -->
+                <origin rpy="1.571 0.21 -0.52" xyz="-0.86 -0.125 -0.05485"/>  <!-- passing the servo rotation mount as 1.57-1.78 = 0.21 -->
                 <axis xyz="1.0 0.0 0.0"/>
             </joint>
@@ -140,5 +154,5 @@
                 <origin rpy="0.0 0.0 0.0" xyz="0.0 0.0 0.0"/>
                 <axis xyz="0.0 0.0 1.0"/>
-                <limits min="-3.14" max="3.14"/>
+                <limits min="-3.1000000" max="3.1000000"/>
             </joint>
                 <!-- fixed joint between thruster and duct -->
@@ -152,5 +166,5 @@
             <actuator name="surge_port_servo" type="servo">
                 <joint name="surge_port_servo2duct_joint"/>
-                <controller position_gain="0.03" velocity_gain="1.0" max_torque="0.2"/>
+                <controller position_gain="0.1" velocity_gain="0.5" max_torque="1.2"/>
             </actuator>
                 <!-- attach thruster/propeller at the thruster link -->
@@ -158,5 +172,5 @@
                 <link name="surge_port_thruster_link"/>
                 <origin rpy="0.0 0.0 0.0" xyz="0.0 0.0 0.0"/>
-                <specs thrust_coeff="0.4472" thrust_coeff_backward="0.3566" torque_coeff="0.01" max_rpm="3000.0"/>
+                <specs thrust_coeff="0.4472" thrust_coeff_backward="0.4472" torque_coeff="0.01" max_rpm="3000.0"/>
                 <propeller diameter="0.08" right="true">
                     <mesh filename="parts/thruster/prop.obj" scale="1.0"/>
@@ -201,5 +215,6 @@
                 <parent name="Vehicle"/>
                 <child name="surge_starboard_servo_link"/>
-                <origin rpy="-1.571 -1.78 0.52" xyz="-0.86 0.125 -0.05485"/>
+                <!-- <origin rpy="-1.571 -1.78 0.52" xyz="-0.86 0.125 -0.05485"/> -->
+                <origin rpy="-1.571 -0.21 0.52" xyz="-0.86 0.125 -0.05485"/>
                 <axis xyz="1.0 0.0 0.0"/>
             </joint>
@@ -210,5 +225,5 @@
                 <origin rpy="0.0 0.0 0.0" xyz="0.0 0.0 0.0"/>
                 <axis xyz="0.0 0.0 1.0"/>
-                <limits min="-3.14" max="3.14"/>
+                <limits min="-3.1000000" max="3.1000000"/>
             </joint>
                 <!-- fixed joint between thruster and duct -->
@@ -222,5 +237,5 @@
             <actuator name="surge_starboard_servo" type="servo">
                 <joint name="surge_starboard_servo2duct_joint"/>
-                <controller position_gain="0.03" velocity_gain="1.0" max_torque="0.2"/>
+                <controller position_gain="0.1" velocity_gain="0.5" max_torque="1.2"/>
             </actuator>
                 <!-- attach thruster/propeller at the thruster link -->
@@ -228,5 +243,5 @@
                 <link name="surge_starboard_thruster_link"/>
                 <origin rpy="0.0 0.0 0.0" xyz="0.0 0.0 0.0"/>
-                <specs thrust_coeff="0.4472" thrust_coeff_backward="0.3566" torque_coeff="0.01" max_rpm="3000.0"/>
+                <specs thrust_coeff="0.4472" thrust_coeff_backward="0.4472" torque_coeff="0.01" max_rpm="3000.0"/>
                 <propeller diameter="0.08" right="true">
                     <mesh filename="parts/thruster/prop.obj" scale="1.0"/>
@@ -248,5 +263,5 @@
                 <specs beam_angle="30.0"/>
                 <range velocity="9.0 9.0 9.0" altitude_min="0.2" altitude_max="200.0"/>
-                <noise velocity="0.01" altitude="0.001"/>
+                <noise velocity="0.005" altitude="0.001"/>
                 <ros_publisher topic="/${robot_name}/dvl/twist" altitude_topic="/${robot_name}/dvl/altitude"/>
             </sensor>
@@ -259,5 +274,5 @@
             <sensor name="gps" type="gps" rate="1.0">
                 <link name="Base"/>
-                <origin rpy="0.0 0.0 0.0" xyz="-0.5 0.0 -0.18"/>
+                <origin rpy="0.0 0.0 0.0" xyz="-0.5 0.0 -0.3"/>
                 <noise ned_position="0.0"/>
                 <ros_publisher topic="/${robot_name}/gps/fix"/>

File: world/ocean_race2.scn.xacro (robot description, xacro)
@@ -15,5 +15,5 @@
         <ocean>
             <water density="1025.0" jerlov="0.2"/>
-            <!-- <waves height="0.0"/> -->
+            <!-- <waves height="0.1"/> -->
             <particles enabled="true"/>
             <current type="uniform">
@@ -32,9 +32,9 @@
     <static name="Bottom" type="model">
         <physical>
-            <mesh filename="objects/flat_terrain.obj" scale="2.0" convex="true"/>
+            <mesh filename="objects/flat_terrain.obj" scale="5.0" convex="true"/>
             <origin xyz="0.0 0.0 0.0" rpy="0.0 0.0 0.0"/>
         </physical>
         <visual>
-            <mesh filename="objects/flat_terrain.obj" scale="2.0"/>
+            <mesh filename="objects/flat_terrain.obj" scale="5.0"/>
             <origin xyz="0.0 0.0 0.0" rpy="0.0 0.0 0.0"/>
         </visual>
