Commit message: update:changing to alpha_rise

File: world/tank.scn.xacro (robot description, xacro)
@@ -9,10 +9,10 @@
 <scenario xmlns:xacro="http://ros.org/wiki/xacro">
     <xacro:arg name="robot_name" default="changeme"/>
-    <xacro:include filename="$(find world_of_stonefish)/vehicles/alpha_std.scn.xacro"/>
-    <xacro:alpha_std robot_name="$(arg robot_name)" xyz="0.0 0.0 0.0" rpy="0.0 0.0 0.0"/>
+    <xacro:include filename="$(find world_of_stonefish)/vehicles/alpha_rise.scn.xacro"/>
+    <xacro:alpha_rise robot_name="$(arg robot_name)" xyz="0.0 0.0 0.0" rpy="0.0 0.0 0.0"/>
     <environment>
-        <ned latitude="41.7777" longitude="3.0333"/>
+        <ned latitude="41" longitude="-71"/>
         <ocean>
-            <water density="1000.0" jerlov="0.2"/>
+            <water density="1031.0" jerlov="0.2"/>
             <waves height="0.0"/>
             <particles enabled="true"/>
@@ -27,10 +27,10 @@
     <static name="tank" type="model">
         <physical>
-            <mesh filename="objects/tank.obj" scale="1.0" convex="false"/>
-            <origin xyz="0.0 0.0 0.0" rpy="0.0 0.0 0.0"/>
+            <mesh filename="objects/tank.obj" scale="0.5" convex="false"/>
+            <origin xyz="0.0 0.0 10" rpy="0.0 0.0 0.0"/>
         </physical>
         <visual>
-            <mesh filename="objects/tank.obj" scale="1.0"/>
-            <origin xyz="0.0 0.0 0.0" rpy="0.0 0.0 0.0"/>
+            <mesh filename="objects/tank.obj" scale="0.5"/>
+            <origin xyz="0.0 0.0 10" rpy="0.0 0.0 0.0"/>
         </visual>
         <material name="Rock"/>
